Commit message: planer draft

File: src/tesseract_env/config/cell.urdf (robot description, URDF)
Before this commit: robot combined, 32 links, 31 joints
Links:
- added link MA1440_tool0
- added link MA2010_tool0
Joints:
- added joint MA1440_joint_6_t-tool0: type fixed, parent MA1440_link_6_t, child MA1440_tool0, origin xyz=0.100 0 0 rpy=0 0 0
- added joint MA2010_joint_6_t-tool0: type fixed, parent MA2010_link_6_t, child MA2010_tool0, origin xyz=0.100 0 0 rpy=0 0 0
